File: hardware/remote-ctrl.sch (KiCad schematic (older format))
At the start: 29 parts, among them IC1 STM32G030K8T6, J1 PRG, J2 CON-1, J3 CON-2, J4 BATT, J5 USB_B_Micro, J6 230AC, K1 AZ850-x, K2 AZ850-x, Q1 PDTC114EU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

Commit message: removed 230VC section, added footprint and components from TME
Parts:
- removed J6: 230AC, symbol Connector:Conn_01x02_Male
- removed PS1: AMEOF10-03S277NZ, Converter_ACDC:Converter_ACDC_RECOM_RAC04-xxSGx_THT, symbol Converter_ACDC:RAC04-3.3SGA
- added C6: 100nF, Capacitor_SMD:C_0805_2012Metric_Pad1.15x1.40mm_HandSolder, symbol Device:C_Small
- added C7: 1uF, Capacitor_SMD:C_0805_2012Metric_Pad1.15x1.40mm_HandSolder, symbol Device:C_Small
- AE1: footprint (none) -> TestPoint:TestPoint_Pad_2.0x2.0mm
- C1, C2, C3: footprint (none) -> Capacitor_SMD:C_0805_2012Metric_Pad1.15x1.40mm_HandSolder
- C4, C5: footprint (none) -> Capacitor_SMD:CP_Elec_4x5.3; TME (none) -> SC1E106M04005VR SAMWHA
- D1, D2: footprint (none) -> Diode_SMD:D_MELF
- D3, D4: footprint (none) -> Diode_SMD:D_1206_3216Metric
- IC1: footprint QFP80P900X900X160-32N -> STM32G030K8T6:QFP80P900X900X160-32N
- J1: footprint (none) -> Connector_PinHeader_2.54mm:PinHeader_1x04_P2.54mm_Vertical
- J2, J3: footprint (none) -> TerminalBlock:TerminalBlock_bornier-3_P5.08mm; TME (none) -> EBBA-03-C-SS-BU
- J4: footprint (none) -> Connector_PinHeader_2.54mm:PinHeader_1x02_P2.54mm_Vertical
- J5: footprint (none) -> Connector_USB:USB_Micro-B_Molex-105017-0001; TME (none) -> 105017-0001 MOLEX
- K1, K2: value AZ850-x -> AZ822-2C-3DSE
- Q1, Q2: footprint (none) -> Package_TO_SOT_SMD:SOT-323_SC-70_Handsoldering
- R1, R2: footprint (none) -> Resistor_SMD:R_0805_2012Metric_Pad1.15x1.40mm_HandSolder
- SW1: value SW_DIP_x03 -> ESD103EZ; footprint (none) -> Button_Switch_SMD:SW_DIP_SPSTx03_Slide_9.78x9.8mm_W8.61mm_P2.54mm
- SW2, SW3: footprint (none) -> Button_Switch_SMD:SW_SPST_Omron_B3FS-101xP; TME (none) -> TACTM-613N-F NINIGI
- U1: value RFM69HW -> RFM69HW-868S2
Connections:
- net GND: now also C6.2, C7.2
- net VDD: now also C6.1, C7.1
- net RF_IRQ: now reaches IC1.12 (PA5)
- net RF_IRQ: now also U1.2 (DIO0)
Other:
- note removed: "230 AV"

Commit message: Added external port, some pin remaped, initial PCB
Parts:
- added J?: EXTERNAL, Connector_PinHeader_2.54mm:PinHeader_1x05_P2.54mm_Vertical, symbol Connector:Conn_01x05_Female
Connections:
- net BTN-1: now also IC1.14 (PA7); no longer IC1.15 (PB0)
- net CODE-1: now also IC1.31 (PB7); no longer IC1.29 (PB5)
- net CODE-3: now also IC1.29 (PB5); no longer IC1.31 (PB7)
- net GND: now also J?.1 (Pin_1)
- net LED-1: now also IC1.10 (PA3); no longer IC1.27 (PB3)
- net LED-2: now also IC1.15 (PB0); no longer IC1.28 (PB4)
- net RF_IRQ: now also IC1.27 (PB3); no longer IC1.12 (PA5)
- net RF_RST: now also IC1.28 (PB4); no longer IC1.7 (PA0)
- net VDD: now also J?.5 (Pin_5)
- net EXT-1: now reaches IC1.1 (PB9)
- net EXT-1: now also J?.4 (Pin_4)
- net EXT-3: now reaches IC1.26 (PA15)
- net EXT-3: now also J?.2 (Pin_2)
- net EXT-2: now reaches IC1.32 (PB8)
- net EXT-2: now also J?.3 (Pin_3)
Changed lines of the file:
@@
 Text Label 6600 3275 0    50   ~ 0
 RF_RST
-Text Label 2425 4225 0    50   ~ 0
+Text Label 3725 2375 3    50   ~ 0
 RF_RST
 Wire Wire Line
-	2425 4225 2725 4225
+	3725 2375 3725 2725
 $Comp
 L Device:Antenna AE1
@@
 Wire Wire Line
 	4025 4925 4025 5200
-Text Label 3925 5200 1    50   ~ 0
+Text Label 3825 5200 1    50   ~ 0
 BTN-1
 Text Label 4025 5200 1    50   ~ 0
@@
 LED-2
 Wire Wire Line
-	3825 2725 3825 2375
-Wire Wire Line
-	3725 2725 3725 2375
-Text Label 3825 2375 3    50   ~ 0
+	3425 4925 3425 5200
+Wire Wire Line
+	3825 4925 3825 5200
+Text Label 3425 5200 1    50   ~ 0
 LED-1
-Text Label 3725 2375 3    50   ~ 0
+Text Label 3925 5200 1    50   ~ 0
 LED-2
 $Comp
@@
 Wire Wire Line
 	3425 2725 3425 2375
-Text Label 3625 2375 3    50   ~ 0
+Text Label 3425 2375 3    50   ~ 0
 CODE-1
 Text Label 3525 2375 3    50   ~ 0
 CODE-2
-Text Label 3425 2375 3    50   ~ 0
+Text Label 3625 2375 3    50   ~ 0
 CODE-3
 $Comp
@@
 RF_IRQ
 Wire Wire Line
-	3625 4925 3625 5200
-Text Label 3625 5200 1    50   ~ 0
+	3825 2725 3825 2375
+Text Label 3825 2375 3    50   ~ 0
 RF_IRQ
 $Comp
@@
 	1    0    0    -1
 $EndComp
+Wire Wire Line
+	2725 3625 2300 3625
+Text Label 2300 3625 0    50   ~ 0
+EXT-1
+Wire Wire Line
+	3325 2725 3325 2375
+Text Label 3325 2375 3    50   ~ 0
+EXT-2
+Wire Wire Line
+	3925 2725 3925 2375
+Text Label 3925 2375 3    50   ~ 0
+EXT-3
+$Comp
+L Connector:Conn_01x05_Female J?
+U 1 1 5F9FDD2B
+P 1425 2275
+F 0 "J?" H 1317 1850 50  0000 C CNN
+F 1 "EXTERNAL" H 1317 1941 50  0000 C CNN
+F 2 "Connector_PinHeader_2.54mm:PinHeader_1x05_P2.54mm_Vertical" H 1425 2275 50  0001 C CNN
+F 3 "~" H 1425 2275 50  0001 C CNN
+	1    1425 2275
+	-1   0    0    1
+$EndComp
+Wire Wire Line
+	1625 2075 1875 2075
+Wire Wire Line
+	1625 2475 1875 2475
+Wire Wire Line
+	1875 2475 1875 2600
+Wire Wire Line
+	1875 2075 1875 1975
+$Comp
+L power:GND #PWR?
+U 1 1 5FA05008
+P 1875 2600
+F 0 "#PWR?" H 1875 2350 50  0001 C CNN
+F 1 "GND" H 1880 2427 50  0000 C CNN
+F 2 "" H 1875 2600 50  0001 C CNN
+F 3 "" H 1875 2600 50  0001 C CNN
+	1    1875 2600
+	1    0    0    -1
+$EndComp
+Wire Wire Line
+	1625 2175 1875 2175
+Wire Wire Line
+	1625 2275 1875 2275
+$Comp
+L power:VDD #PWR?
+U 1 1 5FA05012
+P 1875 1975
+F 0 "#PWR?" H 1875 1825 50  0001 C CNN
+F 1 "VDD" H 1890 2148 50  0000 C CNN
+F 2 "" H 1875 1975 50  0001 C CNN
+F 3 "" H 1875 1975 50  0001 C CNN
+	1    1875 1975
+	1    0    0    -1
+$EndComp
+Wire Wire Line
+	1625 2375 1875 2375
+Text Label 1875 2175 2    50   ~ 0
+EXT-1
+Text Label 1875 2275 2    50   ~ 0
+EXT-2
+Text Label 1875 2375 2    50   ~ 0
+EXT-3
 $EndSCHEMATC

Commit message: Selected elements for BOM
Parts:
- C4, C5: TME SC1E106M04005VR SAMWHA -> GRM319R6YA106KA12D
- D1, D2: value D_Schottky -> TMBAT49FILM
- gave numbers to parts that had none: 1
Changed lines of the file:
@@
 P 2400 5875
 F 0 "D1" H 2400 5658 50  0000 C CNN
-F 1 "D_Schottky" H 2400 5749 50  0000 C CNN
+F 1 "TMBAT49FILM" H 2400 5749 50  0000 C CNN
 F 2 "Diode_SMD:D_MELF" H 2400 5875 50  0001 C CNN
 F 3 "~" H 2400 5875 50  0001 C CNN
@@
 P 5125 5900
 F 0 "D2" H 5125 5683 50  0000 C CNN
-F 1 "D_Schottky" H 5125 5774 50  0000 C CNN
+F 1 "TMBAT49FILM" H 5125 5774 50  0000 C CNN
 F 2 "Diode_SMD:D_MELF" H 5125 5900 50  0001 C CNN
 F 3 "~" H 5125 5900 50  0001 C CNN
+F 4 "" H 5125 5900 50  0001 C CNN "Field4"
 	1    5125 5900
 	-1   0    0    1
@@
 F 2 "Capacitor_SMD:CP_Elec_4x5.3" H 8275 5200 50  0001 C CNN
 F 3 "~" H 8275 5200 50  0001 C CNN
-F 4 "SC1E106M04005VR SAMWHA" H 8275 5200 50  0001 C CNN "TME"
+F 4 "GRM319R6YA106KA12D" H 8275 5200 50  0001 C CNN "TME"
 	1    8275 5200
 	1    0    0    -1
@@
 F 2 "Capacitor_SMD:CP_Elec_4x5.3" H 9250 5200 50  0001 C CNN
 F 3 "~" H 9250 5200 50  0001 C CNN
-F 4 "SC1E106M04005VR SAMWHA" H 9250 5200 50  0001 C CNN "TME"
+F 4 "GRM319R6YA106KA12D" H 9250 5200 50  0001 C CNN "TME"
 	1    9250 5200
 	1    0    0    -1
@@
 EXT-3
 $Comp
-L Connector:Conn_01x05_Female J?
+L Connector:Conn_01x05_Female J6
 U 1 1 5F9FDD2B
 P 1425 2275
-F 0 "J?" H 1317 1850 50  0000 C CNN
+F 0 "J6" H 1317 1850 50  0000 C CNN
 F 1 "EXTERNAL" H 1317 1941 50  0000 C CNN
 F 2 "Connector_PinHeader_2.54mm:PinHeader_1x05_P2.54mm_Vertical" H 1425 2275 50  0001 C CNN
@@
 	1875 2075 1875 1975
 $Comp
-L power:GND #PWR?
+L power:GND #PWR0118
 U 1 1 5FA05008
 P 1875 2600
-F 0 "#PWR?" H 1875 2350 50  0001 C CNN
+F 0 "#PWR0118" H 1875 2350 50  0001 C CNN
 F 1 "GND" H 1880 2427 50  0000 C CNN
 F 2 "" H 1875 2600 50  0001 C CNN
@@
 	1625 2275 1875 2275
 $Comp
-L power:VDD #PWR?
+L power:VDD #PWR0119
 U 1 1 5FA05012
 P 1875 1975
-F 0 "#PWR?" H 1875 1825 50  0001 C CNN
+F 0 "#PWR0119" H 1875 1825 50  0001 C CNN
 F 1 "VDD" H 1890 2148 50  0000 C CNN
 F 2 "" H 1875 1975 50  0001 C CNN
